File: PCB Stack Version A/Bottom.sch (EAGLE design)
At the start: 33 parts, among them U1 ADS1115IDGST, U2 MCP1701AT-5002I/CB

Commit message: PCB Schematics  and boards added
Other:
- note added: "PWR"
- note added: "RP2040-Zero"
Changed lines of the file:
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@@
 <text x="279.4" y="48.26" size="1.778" layer="91">3S</text>
 <text x="279.4" y="45.72" size="1.778" layer="91">4S</text>
+<wire x1="-99.06" y1="81.28" x2="-99.06" y2="15.24" width="0.1524" layer="97"/>
+<wire x1="-99.06" y1="15.24" x2="7.62" y2="15.24" width="0.1524" layer="97"/>
+<wire x1="7.62" y1="15.24" x2="7.62" y2="81.28" width="0.1524" layer="97"/>
+<wire x1="7.62" y1="81.28" x2="-99.06" y2="81.28" width="0.1524" layer="97"/>
+<text x="-93.98" y="76.2" size="2.54" layer="97">PWR</text>
+<text x="53.34" y="50.8" size="5.08" layer="97">RP2040-Zero</text>
 </plain>
 <instances>
